Commit message: added ros2_control

File: myrt_description/urdf/myrt.urdf.xacro (robot description, xacro)
@@ -1,19 +1,19 @@
 <?xml version="1.0" ?>
 <robot name="myrt" xmlns:xacro="http://www.ros.org/wiki/xacro">
-  <xacro:include filename="$(find myrt_bot)/urdf/materials.xacro" />
-<xacro:include filename="$(find myrt_bot)/urdf/ros2_control.xacro" />
-<!-- <xacro:include filename="$(find myrt_bot)/urdf/myrt.trans" /> -->
-<xacro:include filename="$(find myrt_bot)/urdf/myrt.gazebo" />
-<xacro:include filename="$(find myrt_bot)/urdf/camera.xacro" />
+  <xacro:include filename="$(find myrt_description)/urdf/materials.xacro" />
+<xacro:include filename="$(find myrt_description)/urdf/ros2_control.xacro" />
+<xacro:include filename="$(find myrt_description)/urdf/myrt_gazebo.xacro" />
+<xacro:include filename="$(find myrt_description)/urdf/camera.xacro" />
+ <link name="world"/>
 <link name="base_link">
   <inertial>
-    <origin xyz="0.08 0.09249999999999968 0.07996229424977229" rpy="0 0 0"/>
+    <origin xyz="0.08 0.0924 0.0799" rpy="0 0 0"/>
     <mass value="37.199178814539344"/>
-    <inertia ixx="0.185521" iyy="0.158923" izz="0.185637" ixy="0.0" iyz="-0.0" ixz="0.0"/>
+    <inertia ixx="0.1855" iyy="0.1589" izz="0.1856" ixy="0.0" iyz="-0.0" ixz="0.0"/>
   </inertial>
   <visual>
     <origin xyz="0 0 0" rpy="0 0 0"/>
     <geometry>
-      <mesh filename="file://$(find myrt_bot)/meshes/base_link.stl" scale="0.001 0.001 0.001"/>
+      <mesh filename="file://$(find myrt_description)/meshes/base_link.stl" scale="0.001 0.001 0.001"/>
     </geometry>
     <material name="silver"/>
@@ -22,5 +22,5 @@
     <origin xyz="0 0 0" rpy="0 0 0"/>
     <geometry>
-      <mesh filename="file://$(find myrt_bot)/meshes/base_link.stl" scale="0.001 0.001 0.001"/>
+      <mesh filename="file://$(find myrt_description)/meshes/base_link.stl" scale="0.001 0.001 0.001"/>
     </geometry>
   </collision>
@@ -28,6 +28,6 @@
 <link name="rr_link_1">
   <inertial>
-    <origin xyz="-0.010000000000000009 -1.3600232051658168e-15 -6.938893903907228e-18" rpy="0 0 0"/>
-    <mass value="0.6011241193103218"/>
+    <origin xyz="-0.01000 -1.36e-15 -6.938e-18" rpy="0 0 0"/>
+    <mass value="0.6011"/>
     <inertia ixx="0.00037" iyy="0.000205" izz="0.000205" ixy="0.0" iyz="0.0" ixz="0.0"/>
   </inertial>
@@ -35,5 +35,5 @@
     <origin xyz="-0.195 -0.155 -0.015" rpy="0 0 0"/>
     <geometry>
-      <mesh filename="file://$(find myrt_bot)/meshes/rr_link_1.stl" scale="0.001 0.001 0.001"/>
+      <mesh filename="file://$(find myrt_description)/meshes/rr_link_1.stl" scale="0.001 0.001 0.001"/>
     </geometry>
     <material name="silver"/>
@@ -42,5 +42,5 @@
     <origin xyz="-0.195 -0.155 -0.015" rpy="0 0 0"/>
     <geometry>
-      <mesh filename="file://$(find myrt_bot)/meshes/rr_link_1.stl" scale="0.001 0.001 0.001"/>
+      <mesh filename="file://$(find myrt_description)/meshes/rr_link_1.stl" scale="0.001 0.001 0.001"/>
     </geometry>
   </collision>
@@ -48,5 +48,5 @@
 <link name="lf_link_1">
   <inertial>
-    <origin xyz="0.010000000000000002 1.3322676295501878e-15 3.469446951953614e-18" rpy="0 0 0"/>
+    <origin xyz="0.010000000000000002 1.33e-15 3.46e-18" rpy="0 0 0"/>
     <mass value="0.6011241193103217"/>
     <inertia ixx="0.00037" iyy="0.000205" izz="0.000205" ixy="-0.0" iyz="-0.0" ixz="-0.0"/>
@@ -55,5 +55,5 @@
     <origin xyz="0.035 -0.03 -0.015" rpy="0 0 0"/>
     <geometry>
-      <mesh filename="file://$(find myrt_bot)/meshes/lf_link_1.stl" scale="0.001 0.001 0.001"/>
+      <mesh filename="file://$(find myrt_description)/meshes/lf_link_1.stl" scale="0.001 0.001 0.001"/>
     </geometry>
     <material name="silver"/>
@@ -62,5 +62,5 @@
     <origin xyz="0.035 -0.03 -0.015" rpy="0 0 0"/>
     <geometry>
-      <mesh filename="file://$(find myrt_bot)/meshes/lf_link_1.stl" scale="0.001 0.001 0.001"/>
+      <mesh filename="file://$(find myrt_description)/meshes/lf_link_1.stl" scale="0.001 0.001 0.001"/>
     </geometry>
   </collision>
@@ -75,5 +75,5 @@
     <origin xyz="0.035 -0.155 -0.015" rpy="0 0 0"/>
     <geometry>
-      <mesh filename="file://$(find myrt_bot)/meshes/lr_link_1.stl" scale="0.001 0.001 0.001"/>
+      <mesh filename="file://$(find myrt_description)/meshes/lr_link_1.stl" scale="0.001 0.001 0.001"/>
     </geometry>
     <material name="silver"/>
@@ -82,5 +82,5 @@
     <origin xyz="0.035 -0.155 -0.015" rpy="0 0 0"/>
     <geometry>
-      <mesh filename="file://$(find myrt_bot)/meshes/lr_link_1.stl" scale="0.001 0.001 0.001"/>
+      <mesh filename="file://$(find myrt_description)/meshes/lr_link_1.stl" scale="0.001 0.001 0.001"/>
     </geometry>
   </collision>
@@ -95,5 +95,5 @@
     <origin xyz="-0.195 -0.03 -0.015" rpy="0 0 0"/>
     <geometry>
-      <mesh filename="file://$(find myrt_bot)/meshes/rf_link_1.stl" scale="0.001 0.001 0.001"/>
+      <mesh filename="file://$(find myrt_description)/meshes/rf_link_1.stl" scale="0.001 0.001 0.001"/>
     </geometry>
     <material name="silver"/>
@@ -102,9 +102,32 @@
     <origin xyz="-0.195 -0.03 -0.015" rpy="0 0 0"/>
     <geometry>
-      <mesh filename="file://$(find myrt_bot)/meshes/rf_link_1.stl" scale="0.001 0.001 0.001"/>
+      <mesh filename="file://$(find myrt_description)/meshes/rf_link_1.stl" scale="0.001 0.001 0.001"/>
     </geometry>
   </collision>
 </link>
-<joint name="Revolute 2" type="continuous">
+<joint name="virtual_joint" type="fixed">
+        <parent link="world"/>
+        <child link="base_link"/>
+        <origin xyz="1.5 0 0" rpy="0 0 0"/>
+    </joint>
+<joint name="left_front_joint" type="continuous">
+  <origin xyz="-0.035 0.03 0.015" rpy="0 0 0"/>
+  <parent link="base_link"/>
+  <child link="lf_link_1"/>
+  <axis xyz="-1.0 0.0 0.0"/>
+</joint>
+<joint name="left_rear_joint" type="continuous">
+  <origin xyz="-0.035 0.155 0.015" rpy="0 0 0"/>
+  <parent link="base_link"/>
+  <child link="lr_link_1"/>
+  <axis xyz="-1.0 0.0 0.0"/>
+</joint>
+<joint name="right_front_joint" type="continuous">
+  <origin xyz="0.195 0.03 0.015" rpy="0 0 0"/>
+  <parent link="base_link"/>
+  <child link="rf_link_1"/>
+  <axis xyz="1.0 0.0 0.0"/>
+</joint>
+<joint name="right_rear_joint" type="continuous">
   <origin xyz="0.195 0.155 0.015" rpy="0 0 0"/>
   <parent link="base_link"/>
@@ -112,22 +135,4 @@
   <axis xyz="1.0 0.0 0.0"/>
 </joint>
-<joint name="Revolute 3" type="continuous">
-  <origin xyz="-0.035 0.03 0.015" rpy="0 0 0"/>
-  <parent link="base_link"/>
-  <child link="lf_link_1"/>
-  <axis xyz="-1.0 0.0 0.0"/>
-</joint>
-<joint name="Revolute 4" type="continuous">
-  <origin xyz="-0.035 0.155 0.015" rpy="0 0 0"/>
-  <parent link="base_link"/>
-  <child link="lr_link_1"/>
-  <axis xyz="-1.0 0.0 0.0"/>
-</joint>
-<joint name="Revolute 5" type="continuous">
-  <origin xyz="0.195 0.03 0.015" rpy="0 0 0"/>
-  <parent link="base_link"/>
-  <child link="rf_link_1"/>
-  <axis xyz="1.0 0.0 0.0"/>
-</joint>
 <xacro:add_camera parent="base_link"/>
 </robot>

File: myrt_description/urdf/myrt_gazebo.xacro (robot description, xacro)
@@ -2,7 +2,4 @@
 <robot name="myrt" xmlns:xacro="http://www.ros.org/wiki/xacro" >
 <xacro:property name="body_color" value="Gazebo/Silver" />
-<gazebo>
-  <plugin name="control" filename="libgazebo_ros_control.so"/>
-</gazebo>
 <gazebo reference="base_link">
   <material>${body_color}</material>
@@ -36,3 +33,10 @@
   <self_collide>true</self_collide>
 </gazebo>
+<gazebo>
+    <plugin filename="libgazebo_ros2_control.so" name="gazebo_ros2_control">
+      <robot_param>robot_description</robot_param>
+      <robot_param_node>robot_state_publisher</robot_param_node>
+      <parameters>$(find myrt_controller)/config/myrt_controllers.yaml</parameters>
+    </plugin>
+  </gazebo>
 </robot>
