Commit message: Update repo structure and README.MD

File: myrt_description/urdf/myrt.urdf.xacro (robot description, xacro)
@@ -5,5 +5,4 @@
 <xacro:include filename="$(find myrt_description)/urdf/myrt_gazebo.xacro" />
 <xacro:include filename="$(find myrt_description)/urdf/camera.xacro" />
- <link name="world"/>
 <link name="base_link">
   <inertial>
@@ -106,9 +105,4 @@
   </collision>
 </link>
-<joint name="virtual_joint" type="fixed">
-        <parent link="world"/>
-        <child link="base_link"/>
-        <origin xyz="1.5 0 0" rpy="0 0 0"/>
-    </joint>
 <joint name="left_front_joint" type="continuous">
   <origin xyz="-0.035 0.03 0.015" rpy="0 0 0"/>
