Commit message: ros2_control implemented and verified for gz

File: myrt_bot/urdf/myrt.urdf.xacro (robot description, xacro)
@@ -6,4 +6,5 @@
 <xacro:include filename="$(find myrt_bot)/urdf/myrt.gazebo" />
 <xacro:include filename="$(find myrt_bot)/urdf/camera.xacro" />
+<!-- <link name="world"/> -->
 <link name="base_link">
   <inertial>
@@ -106,9 +107,14 @@
   </collision>
 </link>
+<!-- <joint name="virtual_joint" type="fixed">
+  <parent link="world"/>
+  <child link="base_link"/>
+  <origin xyz="0 0 0" rpy="0 0 0"/>
+</joint> -->
 <joint name="Revolute 2" type="continuous">
   <origin xyz="0.195 0.155 0.015" rpy="0 0 0"/>
   <parent link="base_link"/>
   <child link="rr_link_1"/>
-  <axis xyz="1.0 0.0 0.0"/>
+  <axis xyz="-1.0 0.0 0.0"/>
 </joint>
 <joint name="Revolute 3" type="continuous">
@@ -128,5 +134,5 @@
   <parent link="base_link"/>
   <child link="rf_link_1"/>
-  <axis xyz="1.0 0.0 0.0"/>
+  <axis xyz="-1.0 0.0 0.0"/>
 </joint>
 <xacro:add_camera parent="base_link"/>

Commit message: TF_LUNA

File: myrt_bot/urdf/myrt.urdf.xacro (robot description, xacro)
@@ -7,4 +7,5 @@
 <xacro:include filename="$(find myrt_bot)/urdf/myrt.gazebo" />
 <xacro:include filename="$(find myrt_bot)/urdf/camera.xacro" />
+<xacro:include filename="$(find myrt_bot)/urdf/tof.xacro" />
 <!-- <link name="world"/> -->
 <link name="base_link">
@@ -138,3 +139,6 @@
 </joint>
 <xacro:add_camera parent="base_link"/>
+ <xacro:tf_luna_sensor name="tof_sensor" parent="base_link">
+    <origin xyz="0.095 0.21 0.07" rpy="0 0 1.5708"/>
+  </xacro:tf_luna_sensor>
 </robot>

Commit message: loosu ku sukesh

File: myrt_bot/urdf/myrt.urdf.xacro (robot description, xacro)
@@ -8,5 +8,5 @@
 <xacro:include filename="$(find myrt_bot)/urdf/camera.xacro" />
 <xacro:include filename="$(find myrt_bot)/urdf/tof.xacro" />
-<!-- <link name="world"/> -->
+<link name="world"/>
 <link name="base_link">
   <inertial>
@@ -109,9 +109,9 @@
   </collision>
 </link>
-<!-- <joint name="virtual_joint" type="fixed">
+<joint name="virtual_joint" type="fixed">
   <parent link="world"/>
   <child link="base_link"/>
   <origin xyz="0 0 0" rpy="0 0 0"/>
-</joint> -->
+</joint>
 <joint name="Revolute 2" type="continuous">
   <origin xyz="0.195 0.155 0.015" rpy="0 0 0"/>
